Commit message: summit_xl_mico.urdf.xacro unsing summit_xl template

File: summit_xl_mico_description/robots/summit_xl_mico.urdf.xacro (robot description, xacro)
@@ -5,18 +5,78 @@
 	<!-- ***************** -->
 	<!-- First we import all posible elements defined in the urdf.xacro files. All these elements are defined as macro:xacros -->
-	<!-- Import Summit XL base -->
-	<xacro:include filename="$(find summit_xl_description)/robots/summit_xl_nocam.urdf.xacro" />
+	<!-- Import summit XL base elements -->
+	<xacro:include filename="$(find summit_xl_description)/urdf/bases/summit_xl_base.urdf.xacro" />
+	<!-- Import summit XL wheels -->
+	<xacro:include filename="$(find summit_xl_description)/urdf/wheels/rubber_wheel.urdf.xacro" />
+	<!-- Import all available sensors -->
+	<xacro:include filename="$(find robotnik_sensors)/urdf/all_sensors.urdf.xacro" />
 	<!-- Import Mico Arm -->
 	<xacro:include filename="$(find mico_description)/robots/mico_arm.urdf.xacro" />
-	<!-- Gazebo ros control plugins -->
-	<!-- xacro:ros_control/ -->
-    <gazebo>
-      <plugin name="ros_control" filename="libgazebo_ros_control.so">
-        <robotNamespace>/summit_xl_mico</robotNamespace>
-        <robotParam>robot_description</robotParam>
-        <controlPeriod>0.001</controlPeriod>
-	    <robotSimType>gazebo_ros_control/DefaultRobotHWSim</robotSimType>
-      </plugin>
-    </gazebo>
+	<!-- ***************** -->
+	<!-- Global parameters -->
+	<!-- ***************** -->
+	<xacro:property name="PI" value="3.1415926535897931"/>
+	<!-- Wheel parameters -->
+	<xacro:property name="wheel_offset_x" value="0.229" />    <!-- x,y,z in translation from base_link to the center of the wheel -->
+	<xacro:property name="wheel_offset_y" value="0.234" />
+	<xacro:property name="wheel_offset_z" value="0.0" />
+	<!-- Flag to select the high or low quality model -->
+	<xacro:property name="hq" value="true" />
+	<!-- *************** -->
+	<!-- Robots Elements -->
+	<!-- *************** -->
+	<!-- Here we create the robot elements using the xacro:macros imported at the beggining of this file -->
+	<!-- Summit XL base -->
+	<xacro:summit_xl_base name="summit_xl" publish_bf="true" hq="${hq}" />
+	<!-- Gazebo ros control pluggins -->
+	<xacro:ros_control/>
+	<!-- Gazebo skid steering pluggins -->
+	<xacro:skid_steering broadcastOdomTF="1"/>
+	<!-- WHEELS -->
+	<xacro:rubber_wheel name="front_right" parent="base_link" reflect="false" hq="${hq}">
+		<origin xyz="${wheel_offset_x} -${wheel_offset_y} ${wheel_offset_z}" rpy="0 0 0"/>
+	</xacro:rubber_wheel>
+	<xacro:rubber_wheel name="front_left" parent="base_link" reflect="true" hq="${hq}">
+		<origin xyz="${wheel_offset_x} ${wheel_offset_y} ${wheel_offset_z}" rpy="0 0 0"/>
+	</xacro:rubber_wheel>
+	<xacro:rubber_wheel name="back_left" parent="base_link" reflect="true" hq="${hq}">
+		<origin xyz="-${wheel_offset_x} ${wheel_offset_y} ${wheel_offset_z}" rpy="0 0 0"/>
+	</xacro:rubber_wheel>
+	<xacro:rubber_wheel name="back_right" parent="base_link" reflect="false" hq="${hq}">
+		<origin xyz="-${wheel_offset_x} -${wheel_offset_y} ${wheel_offset_z}" rpy="0 0 0"/>
+	</xacro:rubber_wheel>
+	<!-- SENSORS -->
+	<!-- xacro:sensor_hokuyo_utm30lx name="hokuyo" parent="base_link">
+		<origin xyz="0.0 0.0 0.33" rpy="0 0 0"/>
+	</xacro:sensor_hokuyo_utm30lx -->
+<!--
+	<xacro:sensor_hokuyo_urg04lx name="hokuyo1" parent="base_link">
+		<origin xyz="-0.1 0.0 0.33" rpy="0 0 0"/>
+	</xacro:sensor_hokuyo_urg04lx>
+-->
+	<!-- xacro:sensor_axis name="camera" parent="base_link">
+		<origin xyz="0.19 0 0.17" rpy="0 ${15*PI/180} 0"/>
+	</xacro:sensor_axis -->
+	<xacro:sensor_imu name="imu" parent="base_link">
+		<origin xyz="-0.18 0.0 0.170" rpy="0 0 0"/>
+	</xacro:sensor_imu>
+	<xacro:sensor_gps name="gps" parent="base_link">
+		<origin xyz="-0.22 0 0.275" rpy="0 0 0"/>
+	</xacro:sensor_gps>
+<!--
+	<xacro:sensor_asus_xtion_pro name="xtion_pro" parent="base_link">
+		<origin xyz="0.3 0.0 0.3" rpy="0 0 0"/>
+	</xacro:sensor_asus_xtion_pro>
+-->
+<!--
+	<xacro:sensor_kinect name="kinect" parent="base_link">
+		<origin xyz="0.325 0.0 0.16" rpy="0 0 0"/>
+	</xacro:sensor_kinect>
+-->
+<!--
+	<xacro:sensor_fotonic name="fotonic" parent="base_link">
+		<origin xyz="0.3 0.0 0.24" rpy="0 0 0"/>
+	</xacro:sensor_fotonic>
+-->
 	<!-- Fix arm to robot base platform -->
 	<joint
